File: seed3-carrier.kicad_sch (KiCad schematic)
At the start: 33 parts, among them J1 AudioJack2, J2 AudioJack2, J3 5V_IN, J4 DISPLAY_UART, U1 TLV9062IDR

Commit message: Add headphone output with switched line mute and assign footprints
Parts:
- removed C4: 100pF, symbol Device:C_Small
- removed C6: 4.7uF, symbol Device:C_Small
- added C12, C13: 4.7uF, Capacitor_SMD:C_1210_3225Metric_Pad1.33x2.70mm_HandSolder, symbol Device:C_Small
- added C14, C15: 470uF 10V, Capacitor_THT:CP_Radial_D8.0mm_P3.50mm, symbol Device:C_Polarized
- added C16: 1uF, Capacitor_SMD:C_1206_3216Metric_Pad1.33x1.80mm_HandSolder, symbol Device:C_Small
- added C17: 100nF, Capacitor_SMD:C_1206_3216Metric_Pad1.33x1.80mm_HandSolder, symbol Device:C_Small
- added C18: 47uF 10V, Capacitor_THT:CP_Radial_D5.0mm_P2.00mm, symbol Device:C_Polarized
- added J5: SJ1-3535NG, Connector_Audio:Jack_3.5mm_CUI_SJ1-3535NG_Horizontal, symbol Connector_Audio:AudioJack3_SwitchTR
- added R10, R11, R12, R9: 20k, Resistor_SMD:R_1206_3216Metric_Pad1.30x1.75mm_HandSolder, symbol Device:R_Small_US
- added R13, R14: 100, Resistor_SMD:R_1206_3216Metric_Pad1.30x1.75mm_HandSolder, symbol Device:R_Small_US
- added R15, R16: 4.7, Resistor_SMD:R_1206_3216Metric_Pad1.30x1.75mm_HandSolder, symbol Device:R_Small_US
- added RV1: 1M INPUT TRIM, Potentiometer_THT:Potentiometer_Bourns_3296W_Vertical, symbol Device:R_Potentiometer_Small
- added U2: TPA6111A2DR, Package_SO:SOIC-8_3.9x4.9mm_P1.27mm, symbol seed3-carrier:TPA6111A2DR
- C1, C10, C11, C2, C3, C5, C8, C9: footprint (none) -> Capacitor_SMD:C_1206_3216Metric_Pad1.33x1.80mm_HandSolder
- C7: footprint (none) -> Capacitor_SMD:C_1210_3225Metric_Pad1.33x2.70mm_HandSolder
- J1, J2: footprint (none) -> Connector_Audio:Jack_6.35mm_Neutrik_NRJ4HF_Horizontal
- J3: footprint (none) -> Connector_PinHeader_2.54mm:PinHeader_1x02_P2.54mm_Vertical
- J4: footprint (none) -> Connector_PinHeader_2.54mm:PinHeader_1x03_P2.54mm_Vertical
- R1, R2, R3, R4, R6, R7, R8: footprint (none) -> Resistor_SMD:R_1206_3216Metric_Pad1.30x1.75mm_HandSolder
- R5: value 1M -> 10M; footprint (none) -> Resistor_SMD:R_1206_3216Metric_Pad1.30x1.75mm_HandSolder
- RV2, RV3: footprint (none) -> Potentiometer_THT:Potentiometer_Alps_RK09K_Single_Vertical
- TP2, TP4, TP5, TP6, TP7, TP8: footprint (none) -> TestPoint:TestPoint_Pad_D2.0mm
- U1: footprint Package_SO:JEITA_SOIC-8_3.9x4.9mm_P1.27mm -> Package_SO:SOIC-8_3.9x4.9mm_P1.27mm
Connections:
- net +5V: now also C17.1, C18.1, U2.8 (VDD)
- net GND: now also C16.2, C17.2, C18.2, J5.S, R13.2, R14.2, U2.4 (GND), U2.5 (SHDN)
- net VREF: now also RV1.1
- net at J2.T, R4.2: now also R3.1
- net at R1.1: now also RV1.2; no longer C3.2
- net HP_SOURCE: now reaches TP8.1, U1.6 (-), U1.7
- net HP_SOURCE: now also C12.1, C13.1; no longer R3.2
- new net: C14.2, R13.1, R15.1
- new net: C15.2, R14.1, R16.1
- new net: C15.1, R12.2, U2.7 (VOUT2)
- new net: C14.1, R11.2, U2.1 (VOUT1)
- new net: C12.2, R9.1
- new net: C13.2, R10.1
- new net: R10.2, R12.1, U2.6 (IN2-)
- new net: R11.1, R9.2, U2.2 (IN1-)
- new net: C16.1, U2.3 (BYPASS)
- new net: C3.2, RV1.3
- new net HP_L: J5.T, R15.2
- new net HP_R: J5.R, R16.2
- new net LINE_SEND: J5.TN, R3.2
- no-connect marks 30 -> 31
Other:
- note added: "Fed through the headphone driver plugging in headphones to the 1/8" jack mutes the 1/4" jack otherwise audio is passed through LINE_SEND"
- note added: "Gain = -1 per channel (20k / 20k)."
- note added: "HEADPHONE OUTPUT"
- note added: "Mono to both ears / 16-64 ohm headphones"
- note added: "RV1: CW = full level. Turn down for hot pickups/pedals."
- moved on the sheet: C2, C5, J2, R2, R3, R4, R6, TP4, TP8, U1B

Commit message: Replace input trimmer with matching front-panel potentiometers
Parts:
- RV1: value 1M INPUT TRIM -> 1M INPUT LEVEL; footprint Potentiometer_THT:Potentiometer_Bourns_3296W_Vertical -> Potentiometer_THT:Potentiometer_Bourns_PTV09A-1_Single_Vertical; MPN 3296W-1-105LF -> PTV09A-4020F-B105
- RV2, RV3: footprint Potentiometer_THT:Potentiometer_Alps_RK09K_Single_Vertical -> Potentiometer_THT:Potentiometer_Bourns_PTV09A-1_Single_Vertical; MPN (none) -> PTV09A-4020F-B103
Changed lines of the file:
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@@
 		)
 	)
-	(label "GND"
-		(at 332.74 66.04 0)
-		(effects
-			(font
-				(size 1.27 1.27)
-			)
-			(justify left bottom)
-		)
-	)
 	(label "HP_R"
 		(at 397.51 76.2 0)
@@
 			)
 		)
-		(property "Footprint" "Potentiometer_THT:Potentiometer_Alps_RK09K_Single_Vertical"
+		(property "Footprint" "Potentiometer_THT:Potentiometer_Bourns_PTV09A-1_Single_Vertical"
 			(at 127 92.71 0)
 			(hide yes)
@@
 			)
 		)
-		(property "Datasheet" ""
+		(property "Datasheet" "https://www.bourns.com/docs/product-datasheets/ptv09.pdf"
 			(at 127 92.71 0)
 			(hide yes)
@@
 		(pin "1"
 		)
-		(instances
+		(property "MPN" "PTV09A-4020F-B103" (at 127 92.71 0) (hide yes) (effects (font (size 1.27 1.27))))
+(instances
 			(project "seed3-carrier"
 				(path "/94ecceca-f8ce-4e68-9c84-99ac5115dfb9"
@@
 			)
 		)
-		(property "Footprint" "Potentiometer_THT:Potentiometer_Alps_RK09K_Single_Vertical"
+		(property "Footprint" "Potentiometer_THT:Potentiometer_Bourns_PTV09A-1_Single_Vertical"
 			(at 127 123.19 0)
 			(hide yes)
@@
 			)
 		)
-		(property "Datasheet" ""
+		(property "Datasheet" "https://www.bourns.com/docs/product-datasheets/ptv09.pdf"
 			(at 127 123.19 0)
 			(hide yes)
@@
 		(pin "1"
 		)
-		(instances
+		(property "MPN" "PTV09A-4020F-B103" (at 127 123.19 0) (hide yes) (effects (font (size 1.27 1.27))))
+(instances
 			(project "seed3-carrier"
 				(path "/94ecceca-f8ce-4e68-9c84-99ac5115dfb9"
@@
 			)
 		)
-		(property "Value" "1M INPUT TRIM"
+		(property "Value" "1M INPUT LEVEL"
 			(at 78.74 53.34 0)
 			(show_name no)
@@
 			)
 		)
-		(property "Footprint" "Potentiometer_THT:Potentiometer_Bourns_3296W_Vertical"
+		(property "Footprint" "Potentiometer_THT:Potentiometer_Bourns_PTV09A-1_Single_Vertical"
 			(at 64.77 50.8 0)
 			(hide yes)
@@
 			)
 		)
-		(property "Datasheet" "https://www.bourns.com/docs/product-datasheets/3296.pdf"
+		(property "Datasheet" "https://www.bourns.com/docs/product-datasheets/ptv09.pdf"
 			(at 64.77 50.8 0)
 			(hide yes)
@@
 			)
 		)
-		(property "MPN" "3296W-1-105LF"
+		(property "MPN" "PTV09A-4020F-B105"
 			(at 64.77 50.8 0)
 			(hide yes)
@@
 					(unit 1)
 				)
+			)
+		)
+	)
+	(symbol
+		(lib_id "power:GND")
+		(at 332.74 66.04 0)
+		(unit 1)
+		(body_style 1)
+		(exclude_from_sim no)
+		(in_bom yes)
+		(on_board yes)
+		(in_pos_files yes)
+		(dnp no)
+		(property "Reference" "#PWR033"
+			(at 332.74 66.04 0)
+			(hide yes)
+			(show_name no)
+			(do_not_autoplace no)
+			(effects
+				(font
+					(size 1.27 1.27)
+				)
+			)
+		)
+		(property "Value" "GND"
+			(at 332.74 69.84 0)
+			(show_name no)
+			(do_not_autoplace no)
+			(effects
+				(font
+					(size 1.27 1.27)
+				)
+			)
+		)
+		(property "Footprint" ""
+			(at 332.74 66.04 0)
+			(hide yes)
+			(show_name no)
+			(do_not_autoplace no)
+			(effects
+				(font
+					(size 1.27 1.27)
+				)
+			)
+		)
+		(property "Datasheet" ""
+			(at 332.74 66.04 0)
+			(show_name no)
+			(do_not_autoplace no)
+			(effects
+				(font
+					(size 1.27 1.27)
+				)
+			)
+		)
+		(property "Description" ""
+			(at 332.74 66.04 0)
+			(show_name no)
+			(do_not_autoplace no)
+			(effects
+				(font
+					(size 1.27 1.27)
+				)
+			)
+		)
+		(pin "1"
+		)
+		(instances
+			(project "seed3-carrier"
+				(path "/94ecceca-f8ce-4e68-9c84-99ac5115dfb9"
+					(reference "#PWR033")
+					(unit 1)
+				)

Commit message: Save initial PCB placement checkpoint
Capture preliminary component placement and schematic testpoint updates. Placement remains in progress; no copper traces or vias have been routed.
Parts:
- removed TP8: TestPoint, TestPoint:TestPoint_Pad_D2.0mm, symbol Connector:TestPoint
- added TP9: TP_AMP_5V, TestPoint:TestPoint_Pad_D2.0mm, symbol Connector:TestPoint
- TP2: value TestPoint -> TP_AUD_IN
- TP4: value TestPoint -> TP_AUD_OUT
- TP5: value TestPoint -> TP_VREF
- TP6: value TestPoint -> TP_5V
- TP7: value TestPoint -> TP_GND
Connections:
- net +5V: now also TP9.1
Changed lines of the file:
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@@
 	)
 	(junction
+		(at 345.44 43.18)
+		(diameter 0)
+		(color 0 0 0 0)
+	)
+	(junction
 		(at 41.91 149.86)
 		(diameter 0)
@@
 	(wire
 		(pts
-			(xy 345.44 48.26) (xy 345.44 44.45)
+			(xy 345.44 48.26) (xy 345.44 43.18)
 		)
 		(stroke
@@
 	(wire
 		(pts
+			(xy 345.44 43.18) (xy 345.44 38.1)
+		)
+		(stroke
+			(width 0)
+			(type default)
+		)
+	)
+	(wire
+		(pts
 			(xy 387.35 121.92) (xy 387.35 129.54)
 		)
@@
 	)
 	(label "HP_SOURCE"
-		(at 204.47 31.75 0)
+		(at 204.47 29.21 0)
 		(effects
 			(font
@@
 			)
 		)
+		(property "MPN" "PTV09A-4020F-B103"
+			(at 127 92.71 0)
+			(hide yes)
+			(show_name no)
+			(do_not_autoplace no)
+			(effects
+				(font
+					(size 1.27 1.27)
+				)
+			)
+		)
 		(pin "2"
 		)
@@
 		(pin "1"
 		)
-		(property "MPN" "PTV09A-4020F-B103" (at 127 92.71 0) (hide yes) (effects (font (size 1.27 1.27))))
-(instances
+		(instances
 			(project "seed3-carrier"
 				(path "/94ecceca-f8ce-4e68-9c84-99ac5115dfb9"
@@
 	)
 	(symbol
+		(lib_id "Connector:TestPoint")
+		(at 345.44 43.18 270)
+		(mirror x)
+		(unit 1)
+		(body_style 1)
+		(exclude_from_sim no)
+		(in_bom yes)
+		(on_board yes)
+		(in_pos_files yes)
+		(dnp no)
+		(fields_autoplaced yes)
+		(property "Reference" "TP9"
+			(at 350.52 41.9099 90)
+			(show_name no)
+			(do_not_autoplace no)
+			(effects
+				(font
+					(size 1.27 1.27)
+				)
+				(justify left)
+			)
+		)
+		(property "Value" "TP_AMP_5V"
+			(at 350.52 44.4499 90)
+			(show_name no)
+			(do_not_autoplace no)
+			(effects
+				(font
+					(size 1.27 1.27)
+				)
+				(justify left)
+			)
+		)
+		(property "Footprint" "TestPoint:TestPoint_Pad_D2.0mm"
+			(at 345.44 38.1 0)
+			(hide yes)
+			(show_name no)
+			(do_not_autoplace no)
+			(effects
+				(font
+					(size 1.27 1.27)
+				)
+			)
+		)
+		(property "Datasheet" ""
+			(at 345.44 38.1 0)
+			(hide yes)
+			(show_name no)
+			(do_not_autoplace no)
+			(effects
+				(font
+					(size 1.27 1.27)
+				)
+			)
+		)
+		(property "Description" "test point"
+			(at 345.44 43.18 0)
+			(hide yes)
+			(show_name no)
+			(do_not_autoplace no)
+			(effects
+				(font
+					(size 1.27 1.27)
+				)
+			)
+		)
+		(pin "1"
+		)
+		(instances
+			(project "seed3-carrier"
+				(path "/94ecceca-f8ce-4e68-9c84-99ac5115dfb9"
+					(reference "TP9")
+					(unit 1)
+				)
+			)
+		)
+	)
+	(symbol
 		(lib_id "Device:C_Small")
 		(at 76.2 166.37 180)
@@
 			)
 		)
-		(property "Value" "TestPoint"
+		(property "Value" "TP_VREF"
 			(at 83.82 151.6379 0)
 			(show_name no)
@@
 			)
 		)
-		(property "Value" "TestPoint"
+		(property "Value" "TP_GND"
 			(at 46.99 116.0779 0)
 			(show_name no)
@@
 		(fields_autoplaced yes)
 		(property "Reference" "TP4"
-			(at 154.94 27.1781 0)
+			(at 154.94 24.6379 0)
 			(show_name no)
 			(do_not_autoplace no)
@@
 			)
 		)
-		(property "Value" "TestPoint"
-			(at 154.94 24.6381 0)
+		(property "Value" "TP_AUD_OUT"
+			(at 154.94 27.1779 0)
 			(show_name no)
 			(do_not_autoplace no)
@@
 	(symbol
 		(lib_id "power:+5V")
-		(at 345.44 44.45 0)
+		(at 345.44 38.1 0)
 		(unit 1)
 		(body_style 1)
@@
 		(dnp no)
 		(property "Reference" "#PWR024"
-			(at 345.44 44.45 0)
+			(at 345.44 38.1 0)
 			(hide yes)
 			(show_name no)
@@
 		)
 		(property "Value" "+5V"
-			(at 345.44 40.65 0)
+			(at 345.44 34.3 0)
 			(show_name no)
 			(do_not_autoplace no)
@@
 		)
 		(property "Footprint" ""
-			(at 345.44 44.45 0)
+			(at 345.44 38.1 0)
 			(hide yes)
 			(show_name no)
@@
 		)
 		(property "Datasheet" ""
-			(at 345.44 44.45 0)
+			(at 345.44 38.1 0)
 			(show_name no)
 			(do_not_autoplace no)
@@
 		)
 		(property "Description" ""
-			(at 345.44 44.45 0)
+			(at 345.44 38.1 0)
 			(show_name no)
 			(do_not_autoplace no)
@@
 			)
 		)
+		(property "MPN" "PTV09A-4020F-B103"
+			(at 127 123.19 0)
+			(hide yes)
+			(show_name no)
+			(do_not_autoplace no)
+			(effects
+				(font
+					(size 1.27 1.27)
+				)
+			)
+		)
 		(pin "2"
 		)
@@
 		(pin "1"
 		)
-		(property "MPN" "PTV09A-4020F-B103" (at 127 123.19 0) (hide yes) (effects (font (size 1.27 1.27))))
-(instances
+		(instances
 			(project "seed3-carrier"
 				(path "/94ecceca-f8ce-4e68-9c84-99ac5115dfb9"
@@
 			)
 		)
-		(property "Value" "TestPoint"
+		(property "Value" "TP_5V"
 			(at 46.99 86.8679 0)
 			(show_name no)
@@
 			)
 		)
-		(property "Value" "TestPoint"
+		(property "Value" "TP_AUD_IN"
 			(at 110.49 36.0679 0)
 			(show_name no)
@@
 					(unit 1)
 				)
-			)
-		)
-	)
-	(symbol
-		(lib_id "Connector:TestPoint")
-		(at 204.47 29.21 0)
-		(mirror y)
-		(unit 1)
-		(body_style 1)
-		(exclude_from_sim no)
-		(in_bom yes)
-		(on_board yes)
-		(in_pos_files yes)
-		(dnp no)
-		(fields_autoplaced yes)
-		(property "Reference" "TP8"
-			(at 201.93 24.6379 0)
-			(show_name no)
-			(do_not_autoplace no)
-			(effects
-				(font
-					(size 1.27 1.27)
-				)
-				(justify left)
-			)
-		)
-		(property "Value" "TestPoint"
-			(at 201.93 27.1779 0)
-			(show_name no)
-			(do_not_autoplace no)
-			(effects
-				(font
-					(size 1.27 1.27)
-				)
-				(justify left)
-			)
-		)
-		(property "Footprint" "TestPoint:TestPoint_Pad_D2.0mm"
-			(at 199.39 29.21 0)
-			(hide yes)
-			(show_name no)
-			(do_not_autoplace no)
-			(effects
-				(font
-					(size 1.27 1.27)
-				)
-			)
-		)
-		(property "Datasheet" ""
-			(at 199.39 29.21 0)
-			(hide yes)
-			(show_name no)
-			(do_not_autoplace no)
-			(effects
-				(font
-					(size 1.27 1.27)
-				)
-			)
-		)
-		(property "Description" "test point"
-			(at 204.47 29.21 0)
-			(hide yes)
-			(show_name no)
-			(do_not_autoplace no)
-			(effects
-				(font
-					(size 1.27 1.27)
-				)
-			)
-		)
-		(pin "1"
-		)
-		(instances
-			(project "seed3-carrier"
-				(path "/94ecceca-f8ce-4e68-9c84-99ac5115dfb9"
-					(reference "TP8")
-					(unit 1)
-				)

Commit message: Save PCB routing progress and Seed3 breakout headers
Parts:
- removed TP2: TP_AUD_IN, TestPoint:TestPoint_Pad_D2.0mm, symbol Connector:TestPoint
- removed TP4: TP_AUD_OUT, TestPoint:TestPoint_Pad_D2.0mm, symbol Connector:TestPoint
- removed TP6: TP_5V, TestPoint:TestPoint_Pad_D2.0mm, symbol Connector:TestPoint
- removed TP7: TP_GND, TestPoint:TestPoint_Pad_D2.0mm, symbol Connector:TestPoint
- added J6: Seed3_PINS_RIGHT, Connector_PinSocket_2.54mm:PinSocket_1x20_P2.54mm_Vertical, symbol Connector:Conn_01x20_Socket
- added J7: Seed3_PINS_LEFT, Connector_PinSocket_2.54mm:PinSocket_1x20_P2.54mm_Vertical, symbol Connector:Conn_01x20_Socket
Connections:
- net +5V: now also J7.19 (Pin_19)
- net 3V3_A: now also J7.1 (Pin_1)
- net DISPLAY_UART_RX: now also J6.6 (Pin_6)
- net DISPLAY_UART_TX: now also J6.7 (Pin_7)
- net GND: now also J6.1 (Pin_1), J7.20 (Pin_20)
- net TONE_POT: now also J7.3 (Pin_3)
- net VOLUME_POT: now also J7.2 (Pin_2)
- net D0: now reaches A1.1 (USB_ID)
- net D0: now also J6.20 (Pin_20)
- net D9: now reaches A1.10 (SPI1_POCI)
- net D9: now also J6.11 (Pin_11)
- net D10: now reaches A1.11 (SPI1_PICO)
- net D10: now also J6.10 (Pin_10)
- net D11: now reaches A1.12 (I2C1_SCL)
- net D11: now also J6.9 (Pin_9)
- net D12: now reaches A1.13 (I2C1_SDA)
- net D12: now also J6.8 (Pin_8)
- net AUDIO_IN_2: now reaches A1.17 (AUDIO_IN_2)
- net AUDIO_IN_2: now also J6.4 (Pin_4)
- net AUDIO_OUT_2: now reaches A1.19 (AUDIO_OUT_2)
- net AUDIO_OUT_2: now also J6.2 (Pin_2)
- net D1: now reaches A1.2 (SD_DATA_3)
- net D1: now also J6.19 (Pin_19)
- net A2: now reaches A1.24 (ADC_2)
- net A2: now also J7.4 (Pin_4)
- net A3: now reaches A1.25 (ADC_3)
- net A3: now also J7.5 (Pin_5)
- net A4: now reaches A1.26 (ADC_4)
- net A4: now also J7.6 (Pin_6)
- net A5: now reaches A1.27 (ADC_5)
- net A5: now also J7.7 (Pin_7)
- net A6: now reaches A1.28 (ADC_6)
- net A6: now also J7.8 (Pin_8)
- net A7: now reaches A1.29 (DAC_OUT2)
- net A7: now also J7.9 (Pin_9)
- net D2: now reaches A1.3 (SD_DATA_2)
- net D2: now also J6.18 (Pin_18)
- net A8: now reaches A1.30 (DAC_OUT1)
- net A8: now also J7.10 (Pin_10)
- net A9: now reaches A1.31 (SAI2_MCLK)
- net A9: now also J7.11 (Pin_11)
- net A10: now reaches A1.32 (SAI2_SD_B)
- net A10: now also J7.12 (Pin_12)
- net D26: now reaches A1.33 (SAI2_SD_A)
- net D26: now also J7.13 (Pin_13)
- net D27: now reaches A1.34 (SAI2_FS)
- net D27: now also J7.14 (Pin_14)
- net A11: now reaches A1.35 (SAI2_SCK)
- net A11: now also J7.15 (Pin_15)
- net USB_D-: now reaches A1.36 (USB_D_-)
- net USB_D-: now also J7.16 (Pin_16)
- net USB_D+: now reaches A1.37 (USB_D_+)
- net USB_D+: now also J7.17 (Pin_17)
- net 3V3_D: now reaches A1.38 (3V3_D)
- net 3V3_D: now also J7.18 (Pin_18)
- net D3: now reaches A1.4 (SD_DATA_1)
- net D3: now also J6.17 (Pin_17)
- net D4: now reaches A1.5 (SD_DATA_0)
- net D4: now also J6.16 (Pin_16)
- net D5: now reaches A1.6 (SD_CMD)
- net D5: now also J6.15 (Pin_15)
- net D6: now reaches A1.7 (SD_CLK)
- net D6: now also J6.14 (Pin_14)
- net D7: now reaches A1.8 (SPI1_CS)
- net D7: now also J6.13 (Pin_13)
- net D8: now reaches A1.9 (SPI1_SCK)
- net D8: now also J6.12 (Pin_12)
- net AUDIO_IN renamed AUDIO_IN_1
- net AUDIO_IN_1: now also J6.5 (Pin_5)
- net AUDIO_OUT renamed AUDIO_OUT_1
- net AUDIO_OUT_1: now also J6.3 (Pin_3)
- no-connect marks 31 -> 1

Commit message: Add reverse-polarity protection and switched input mute
Parts:
- added Q1: AO3401A, Package_TO_SOT_SMD:SOT-23, symbol Transistor_FET:AO3401A
- J1: value AudioJack2 -> AudioJack2_Switch; symbol Connector_Audio:AudioJack2 -> Connector_Audio:AudioJack2_Switch
Connections:
- net +5V: now also Q1.2 (S); no longer J3.1 (Pin_1)
- net GND: now also J1.TN, Q1.1 (G)
- new net: J3.1 (Pin_1), Q1.3 (D)
- no-connect marks 1 -> 2
Other:
- note added: "MOSFET is reverse polarity protection"
- note added: "OPAMP power rails"
- moved on the sheet: C9, J3
