File: seed3-carrier.kicad_sch (KiCad schematic)
At the start: 48 parts, among them J1 AudioJack2_Switch, J2 AudioJack2, J3 5V_IN, J4 DISPLAY_UART, J5 SJ1-3535NG, J6 Seed3_PINS_RIGHT, J7 Seed3_PINS_LEFT, Q1 AO3401A, U1 TLV9062IDR, U2 TPA6111A2DR

Commit message: Expand display header to four pins with protected 5V
Preserve GND and UART pin assignments and add protected +5V on pin 4. Reposition and label the header, reroute UART connections, and complete the power route with a short bottom-layer crossing beneath the buffered audio input. Refill copper zones.
Parts:
- J4: footprint Connector_PinHeader_2.54mm:PinHeader_1x03_P2.54mm_Vertical -> Connector_PinHeader_2.54mm:PinHeader_1x04_P2.54mm_Vertical; symbol Connector_Generic:Conn_01x03 -> Connector_Generic:Conn_01x04
Connections:
- net +5V: now also J4.4 (Pin_4)
Changed lines of the file:
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@@
 	)
 	(symbol
-		(lib_id "Connector_Generic:Conn_01x03")
+		(lib_id "Connector_Generic:Conn_01x04")
 		(at 134.62 154.94 0)
 		(mirror x)
@@
 			)
 		)
-		(property "Footprint" "Connector_PinHeader_2.54mm:PinHeader_1x03_P2.54mm_Vertical"
+		(property "Footprint" "Connector_PinHeader_2.54mm:PinHeader_1x04_P2.54mm_Vertical"
 			(at 134.62 154.94 0)
 			(hide yes)
@@
 			)
 		)
-		(property "Description" "Generic connector, single row, 01x03, script generated (kicad-library-utils/schlib/autogen/connector/)"
+		(property "Description" "Generic connector, single row, 01x04, script generated (kicad-library-utils/schlib/autogen/connector/)"
 			(at 134.62 154.94 0)
 			(hide yes)
@@
 		(pin "3"
 		)
+		(pin "4")
 		(instances
 			(project "seed3-carrier"
@@
 	)
 	(embedded_fonts no)
+	(wire (pts (xy 129.54 149.86) (xy 121.92 149.86))
+		(stroke (width 0) (type default)))
+	(label "+5V" (at 121.92 149.86 0)
+		(effects (font (size 1.27 1.27)) (justify left bottom)))
 )

Commit message: Finalize potentiometer mounts and fabrication purchasing package
Parts:
- RV1, RV2, RV3: footprint Potentiometer_THT:Potentiometer_Bourns_PTV09A-1_Single_Vertical -> Seed3_Carrier:Potentiometer_Bourns_PTV09A-4_Single_Vertical_3mmMount
Changed lines of the file:
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@@
 			)
 		)
-		(property "Footprint" "Potentiometer_THT:Potentiometer_Bourns_PTV09A-1_Single_Vertical"
+		(property "Footprint" "Seed3_Carrier:Potentiometer_Bourns_PTV09A-4_Single_Vertical_3mmMount"
 			(at 127 92.71 0)
 			(hide yes)
@@
 			)
 		)
-		(property "Footprint" "Potentiometer_THT:Potentiometer_Bourns_PTV09A-1_Single_Vertical"
+		(property "Footprint" "Seed3_Carrier:Potentiometer_Bourns_PTV09A-4_Single_Vertical_3mmMount"
 			(at 127 123.19 0)
 			(hide yes)
@@
 			)
 		)
-		(property "Footprint" "Potentiometer_THT:Potentiometer_Bourns_PTV09A-1_Single_Vertical"
+		(property "Footprint" "Seed3_Carrier:Potentiometer_Bourns_PTV09A-4_Single_Vertical_3mmMount"
 			(at 64.77 50.8 0)
 			(hide yes)
